File: kicad/kicad.kicad_sch (KiCad schematic)
At the start: 22 parts

Commit message: updated
Parts:
- removed R?: 100, symbol Device:R
- added D?: (no value), symbol Diode:1N4005
- added J? (x2): (no value), symbol Connector:Conn_01x01_Female
- added R? (x2): 100, symbol Device:R
- added U? (x2): (no value), symbol Analog_Switch:MAX313CPE
- added U?: (no value), symbol Isolator:TLP785
- C?: value (none) -> 10µF
- C?: value (none) -> 0.1nF
Connections:
- net Analog Audio (L): now also U?.15; no longer U?.10
- net Analog Audio (R): now also U?.10; no longer U?.6
- net Analog Video: now also U?.6; no longer U?.2
- net GND: now also U?.2, U?.4 (V-), U?.5 (GND)
- net GNDA: now also U?.3; no longer J?.4, J?.4
- net Output Enabled?: now also U?.9 (PA4), D?.1 (K); no longer R?.1, R?.2, U?.1, U?.8, U?.8 (PA5), U?.9
- net VCC: now also Q?.1 (C), U?.12 (VL), U?.13 (V+)
- net at Q?.3 (E): now also R?.1, R?.2; no longer D?.2 (A)
- net at J?.1 (In): now also U?.7; no longer U?.3
- net at J?.1 (In): now also U?.14; no longer U?.11
- net at J?.1 (In): now also U?.11; no longer U?.7
- new net: D?.2 (A), R?.2
- new net: J?.1 (Pin_1), U?.3
- new net: D?.2 (A), R?.1, R?.2, U?.1, U?.16, U?.8, U?.8 (PA5), U?.9
- new net: J?.1 (Pin_1), U?.4
- new net: R?.1, U?.1
- new net Analog GND: J?.4, J?.4, U?.2
Other:
- note removed: "*Funktionsweiße:* Der Microkontroller lauscht über die Serial verbindung auf Daten. Matchen die ersten 4 bits bei dem epfangen byte mit der eingestellten Adresse, wird "Output Enabled" nach einem kleinen delay auf "high" geschaltet¹. Sollte dies nicht der fall sein, und die Adresse nicht übereinstimmen wird "Output Enabled" auf "low" gezogen. "Output Enabled" = High: Das anliegende Analog signal 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"
- moved on the sheet: C?, D?, J?, Q?, R?, SW?, U?, U?A, U?B, U?C
